File: MadCat/386/386.kicad_pcb (KiCad board)
At the start: 0 parts

Commit message: Update
Parts:
- added H1: HOLE1, mad5150:HOLE, F.Cu at (56.3, 31.5)
- added H2: HOLE1, mad5150:HOLE, F.Cu at (56.3, 148.3)
- added H3: HOLE1, mad5150:HOLE, F.Cu at (56.3, 224.5)
- added H5: HOLE1, mad5150:HOLE, F.Cu at (199.2, 148.3)
- added H6: HOLE1, mad5150:HOLE, F.Cu at (199.2, 224.5)
- added H7: HOLE1, mad5150:HOLE, F.Cu at (346.5, 31.5)
- added H8: HOLE1, mad5150:HOLE, F.Cu at (346.5, 148.3)
- added H9: HOLE1, mad5150:HOLE, F.Cu at (346.5, 224.5)
Other:
- board outline added: 304.8 x 215.9 mm
- copper layers 0 -> 2
