File: MadCat/386/386.kicad_pcb (KiCad board)
At the start: 2 copper layers, 304.8 x 215.9 mm, 8 parts

Commit message: Update
Parts:
- added C1: 47pF, Capacitor_THT:C_Disc_D7.0mm_W2.5mm_P5.00mm, F.Cu at (-23.7, 11.3)
- added C100: 10pF, Capacitor_THT:C_Disc_D7.0mm_W2.5mm_P5.00mm, F.Cu at (-23.7, 31.6)
- added C101: 0.047uF, Capacitor_THT:C_Disc_D7.0mm_W2.5mm_P5.00mm, F.Cu at (-23.7, 35.6)
- added C114: 47pF, Capacitor_THT:C_Disc_D7.0mm_W2.5mm_P5.00mm, F.Cu at (-23.7, 39.7)
- added C117: 18pF, Capacitor_THT:C_Disc_D7.0mm_W2.5mm_P5.00mm, F.Cu at (-23.7, 43.7)
- added C19: 10uF, Capacitor_THT:CP_Radial_D4.0mm_P2.00mm, F.Cu at (-70.1, 129.6)
- added C2: 47pF, Capacitor_THT:C_Disc_D7.0mm_W2.5mm_P5.00mm, F.Cu at (-23.7, 15.4)
- added C60: 47pF, Capacitor_THT:C_Disc_D7.0mm_W2.5mm_P5.00mm, F.Cu at (-23.7, 19.4)
- added C9: 10uF, Capacitor_THT:CP_Radial_D4.0mm_P2.00mm, F.Cu at (-70.1, 124.0)
- added C97: 0.001uF, Capacitor_THT:C_Disc_D7.0mm_W2.5mm_P5.00mm, F.Cu at (-23.7, 23.5)
- added C98: 0.047uF, Capacitor_THT:C_Disc_D7.0mm_W2.5mm_P5.00mm, F.Cu at (-23.7, 27.5)
- added CR1: 1N914, Diode_THT:D_DO-35_SOD27_P7.62mm_Horizontal, F.Cu at (-31.9, 71.6)
- added CR2: 1N914, Diode_THT:D_DO-35_SOD27_P7.62mm_Horizontal, F.Cu at (-31.9, 75.2)
- added CR3: 1N914, Diode_THT:D_DO-35_SOD27_P7.62mm_Horizontal, F.Cu at (-31.9, 78.7)
- added E123: Conn_01x09_Pin, Connector_PinHeader_2.54mm:PinHeader_1x09_P2.54mm_Vertical, F.Cu at (-56.8, 113.2)
- added ER1: Conn_01x09_Pin, Connector_PinHeader_2.54mm:PinHeader_1x09_P2.54mm_Vertical, F.Cu at (-52.2, 113.2)
- added ER2: Conn_01x09_Pin, Connector_PinHeader_2.54mm:PinHeader_1x09_P2.54mm_Vertical, F.Cu at (-47.6, 113.2)
- added F2: F 5A, Fuse:Fuse_1206_3216Metric, F.Cu at (-62.6, 117.1)
- added H2: KEYLOCK, Connector_PinHeader_2.54mm:PinHeader_1x02_P2.54mm_Vertical, F.Cu at (-64.0, 123.6)
- added J115: SPEAKER, Connector_PinHeader_2.54mm:PinHeader_1x04_P2.54mm_Vertical, F.Cu at (-69.6, 105.6)
- added J116: KEYBOARD, Connector_PinHeader_2.54mm:PinHeader_1x07_P2.54mm_Vertical, F.Cu at (-20.4, 84.0)
- added J118: BATTERY, Connector_PinHeader_2.54mm:PinHeader_1x04_P2.54mm_Vertical, F.Cu at (-65.0, 105.6)
- added L1: FerriteBead, Inductor_SMD:L_Panasonic_PCC-M0850M, F.Cu at (-52.1, 67.9)
- added L2: FerriteBead, Inductor_SMD:L_Panasonic_PCC-M0850M, F.Cu at (-52.1, 77.5)
- added L3: FerriteBead, Inductor_SMD:L_Panasonic_PCC-M0850M, F.Cu at (-52.1, 87.0)
- added L4: FerriteBead, Inductor_SMD:L_Panasonic_PCC-M0850M, F.Cu at (-52.1, 96.6)
- added L6: FerriteBead, Inductor_SMD:L_Panasonic_PCC-M0850M, F.Cu at (-52.1, 106.1)
- added MRB4: 33R, Resistor_THT:R_Array_SIP9, F.Cu at (-57.0, 48.5)
- added MRP1: 33R, Package_DIP:DIP-20_W7.62mm_Socket_LongPads, F.Cu at (-43.1, 105.8)
- added MRP5: 4K7, Resistor_THT:R_Array_SIP10, F.Cu at (-96.9, 105.4)
- added MRP6: 8K2, Resistor_THT:R_Array_SIP11, F.Cu at (-96.9, 101.2)
- added MRP7: 4K7, Resistor_THT:R_Array_SIP10, F.Cu at (-96.9, 109.5)
- added MRP8: 4K7, Resistor_THT:R_Array_SIP10, F.Cu at (-96.9, 113.7)
- added MRP9: 4K7, Resistor_THT:R_Array_SIP10, F.Cu at (-96.9, 117.9)
- added MU31: 51256-10, Package_DIP:DIP-16_W7.62mm, F.Cu at (-31.9, 83.7)
- added Q1: TL431LP, Package_TO_SOT_THT:TO-92_Inline, F.Cu at (-69.9, 118.7)
- added R1: 87K, Resistor_THT:R_Axial_DIN0207_L6.3mm_D2.5mm_P10.16mm_Horizontal, F.Cu at (-97.5, 48.5)
- added R10: 180R, Resistor_THT:R_Axial_DIN0207_L6.3mm_D2.5mm_P10.16mm_Horizontal, F.Cu at (-97.5, 72.8)
- added R1000: 20K, Resistor_THT:R_Axial_DIN0207_L6.3mm_D2.5mm_P10.16mm_Horizontal, F.Cu at (-70.8, 84.9)
- added R12: 1K, Resistor_THT:R_Axial_DIN0207_L6.3mm_D2.5mm_P10.16mm_Horizontal, F.Cu at (-97.5, 76.8)
- added R13: 180R, Resistor_THT:R_Axial_DIN0207_L6.3mm_D2.5mm_P10.16mm_Horizontal, F.Cu at (-97.5, 80.9)
- added R14: 20K, Resistor_THT:R_Axial_DIN0207_L6.3mm_D2.5mm_P10.16mm_Horizontal, F.Cu at (-97.5, 84.9)
- added R15: 8K2, Resistor_THT:R_Axial_DIN0207_L6.3mm_D2.5mm_P10.16mm_Horizontal, F.Cu at (-97.5, 89.0)
- added R16: 1K, Resistor_THT:R_Axial_DIN0207_L6.3mm_D2.5mm_P10.16mm_Horizontal, F.Cu at (-97.5, 93.0)
- added R17: 22M, Resistor_THT:R_Axial_DIN0207_L6.3mm_D2.5mm_P10.16mm_Horizontal, F.Cu at (-97.5, 97.1)
- added R18: 180R, Resistor_THT:R_Axial_DIN0207_L6.3mm_D2.5mm_P10.16mm_Horizontal, F.Cu at (-84.2, 48.5)
- added R19: 470K, Resistor_THT:R_Axial_DIN0207_L6.3mm_D2.5mm_P10.16mm_Horizontal, F.Cu at (-84.2, 52.5)
- added R2: 48K, Resistor_THT:R_Axial_DIN0207_L6.3mm_D2.5mm_P10.16mm_Horizontal, F.Cu at (-97.5, 52.5)
- added R20: 1K, Resistor_THT:R_Axial_DIN0207_L6.3mm_D2.5mm_P10.16mm_Horizontal, F.Cu at (-84.2, 56.6)
- added R21: 1K, Resistor_THT:R_Axial_DIN0207_L6.3mm_D2.5mm_P10.16mm_Horizontal, F.Cu at (-84.2, 60.6)
- added R22: 8K2, Resistor_THT:R_Axial_DIN0207_L6.3mm_D2.5mm_P10.16mm_Horizontal, F.Cu at (-84.2, 64.7)
- added R24: 1K, Resistor_THT:R_Axial_DIN0207_L6.3mm_D2.5mm_P10.16mm_Horizontal, F.Cu at (-84.2, 68.7)
- added R25: 30R, Resistor_THT:R_Axial_DIN0207_L6.3mm_D2.5mm_P10.16mm_Horizontal, F.Cu at (-84.2, 72.8)
- added R26: 30R, Resistor_THT:R_Axial_DIN0207_L6.3mm_D2.5mm_P10.16mm_Horizontal, F.Cu at (-84.2, 76.8)
- added R28/9: 180R, Resistor_THT:R_Axial_DIN0207_L6.3mm_D2.5mm_P10.16mm_Horizontal, F.Cu at (-70.8, 89.0)
- added R3: 270R, Resistor_THT:R_Axial_DIN0207_L6.3mm_D2.5mm_P10.16mm_Horizontal, F.Cu at (-97.5, 56.6)
- added R30: 180R, Resistor_THT:R_Axial_DIN0207_L6.3mm_D2.5mm_P10.16mm_Horizontal, F.Cu at (-84.2, 80.9)
- added R31: 68R, Resistor_THT:R_Axial_DIN0207_L6.3mm_D2.5mm_P10.16mm_Horizontal, F.Cu at (-84.2, 84.9)
- added R33: 68R, Resistor_THT:R_Axial_DIN0207_L6.3mm_D2.5mm_P10.16mm_Horizontal, F.Cu at (-84.2, 89.0)
- added R34: 22R, Resistor_THT:R_Axial_DIN0207_L6.3mm_D2.5mm_P10.16mm_Horizontal, F.Cu at (-84.2, 93.0)
- added R35: 22R, Resistor_THT:R_Axial_DIN0207_L6.3mm_D2.5mm_P10.16mm_Horizontal, F.Cu at (-84.2, 97.1)
- added R36: 68R, Resistor_THT:R_Axial_DIN0207_L6.3mm_D2.5mm_P10.16mm_Horizontal, F.Cu at (-70.8, 48.5)
- added R37: 51R, Resistor_THT:R_Axial_DIN0207_L6.3mm_D2.5mm_P10.16mm_Horizontal, F.Cu at (-70.8, 52.5)
- added R38: 68R, Resistor_THT:R_Axial_DIN0207_L6.3mm_D2.5mm_P10.16mm_Horizontal, F.Cu at (-70.8, 56.6)
- added R39: 10K, Resistor_THT:R_Axial_DIN0207_L6.3mm_D2.5mm_P10.16mm_Horizontal, F.Cu at (-70.8, 60.6)
- added R4: 4K7, Resistor_THT:R_Axial_DIN0207_L6.3mm_D2.5mm_P10.16mm_Horizontal, F.Cu at (-97.5, 60.6)
- added R40: 10K, Resistor_THT:R_Axial_DIN0207_L6.3mm_D2.5mm_P10.16mm_Horizontal, F.Cu at (-70.8, 64.7)
- added R41: 20K, Resistor_THT:R_Axial_DIN0207_L6.3mm_D2.5mm_P10.16mm_Horizontal, F.Cu at (-70.8, 68.7)
- added R42: 180R, Resistor_THT:R_Axial_DIN0207_L6.3mm_D2.5mm_P10.16mm_Horizontal, F.Cu at (-70.8, 72.8)
- added R44: 60R, Resistor_THT:R_Axial_DIN0207_L6.3mm_D2.5mm_P10.16mm_Horizontal, F.Cu at (-70.8, 76.8)
- added R5: 1K, Resistor_THT:R_Axial_DIN0207_L6.3mm_D2.5mm_P10.16mm_Horizontal, F.Cu at (-97.5, 64.7)
- added R8: 30R, Resistor_THT:R_Axial_DIN0207_L6.3mm_D2.5mm_P10.16mm_Horizontal, F.Cu at (-97.5, 68.7)
- added R999: 20K, Resistor_THT:R_Axial_DIN0207_L6.3mm_D2.5mm_P10.16mm_Horizontal, F.Cu at (-70.8, 80.9)
- added RB4: 33R, Resistor_THT:R_Array_SIP9, F.Cu at (-57.0, 52.7)
- added RP3: 8K2, Resistor_THT:R_Array_SIP10, F.Cu at (-96.9, 122.0)
- added RP4: 8K2, Resistor_THT:R_Array_SIP10, F.Cu at (-96.9, 126.2)
- added RP5: 8K2, Resistor_THT:R_Array_SIP10, F.Cu at (-96.9, 130.4)
- added RP6: 8K2, Resistor_THT:R_Array_SIP9, F.Cu at (-57.0, 56.9)
- added RP7: 20K, Resistor_THT:R_Array_SIP10, F.Cu at (-96.9, 134.5)
- added RP8: 8K2, Resistor_THT:R_Array_SIP9, F.Cu at (-57.0, 61.0)
- added RX1: 20K, Resistor_THT:R_Axial_DIN0207_L6.3mm_D2.5mm_P10.16mm_Horizontal, F.Cu at (-70.8, 93.0)
- added RX2: 20K, Resistor_THT:R_Axial_DIN0207_L6.3mm_D2.5mm_P10.16mm_Horizontal, F.Cu at (-70.8, 97.1)
- added SW1: SW_DIP_x08, Button_Switch_THT:SW_DIP_SPSTx08_Slide_9.78x22.5mm_W7.62mm_P2.54mm, F.Cu at (-31.5, 106.9)
- added U1: 8259A-2, Package_DIP:DIP-28_W15.24mm, F.Cu at (-152.6, 11.4)
- added U12: 2764, Package_DIP:DIP-28_W15.24mm, F.Cu at (-115.9, 11.4)
- added U13: 2764, Package_DIP:DIP-28_W15.24mm, F.Cu at (-97.5, 11.4)
- added U14: 2764, Package_DIP:DIP-28_W15.24mm, F.Cu at (-79.1, 11.4)
- added U15: 2764, Package_DIP:DIP-28_W15.24mm, F.Cu at (-60.7, 11.4)
- added U2: 8259A-2, Package_DIP:DIP-28_W15.24mm, F.Cu at (-134.2, 11.4)
- added U22: 8237A, Package_DIP:DIP-40_W15.24mm, F.Cu at (-152.6, 80.5)
- added U23: 8237A, Package_DIP:DIP-40_W15.24mm, F.Cu at (-134.2, 80.5)
- added U30: 74LS612, Package_DIP:DIP-40_W15.24mm, F.Cu at (-115.9, 80.5)
- added U44: 8254, Package_DIP:DIP-24_W15.24mm, F.Cu at (-152.6, 48.5)
- added U45: 8254, Package_DIP:DIP-24_W15.24mm, F.Cu at (-134.2, 48.5)
- added U69: 74F74, Package_DIP:DIP-28_W15.24mm, F.Cu at (-42.3, 11.4)
- added U77: MC146818, Package_DIP:DIP-24_W15.24mm, F.Cu at (-115.9, 48.5)
- added U89: 74F175BB, Package_DIP:DIP-16_W7.62mm_Socket_LongPads, F.Cu at (-43.1, 83.8)
- added U91: 74ALS1035, Package_SO:SOIC-14_3.9x8.7mm_P1.27mm, F.Cu at (-30.3, 51.7)
- added U92: 74F11, Package_SO:SOIC-14_3.9x8.7mm_P1.27mm, F.Cu at (-21.9, 51.7)
- added U93: SN75477, Package_DIP:DIP-8_W7.62mm_Socket_LongPads, F.Cu at (-43.1, 71.9)
- added Y2: 32.76KHz, Crystal:Crystal_HC49-U_Vertical, F.Cu at (-41.1, 66.5)
