File: MadCat/386/386.kicad_sch (KiCad schematic)
At the start: 207 parts, among them J101 32 Bit Mem Connector, J102 Bus_ISA_16bit, J115 SPEAKER, J116 KEYBOARD, J118 BATTERY, P101 Conn_01x80_Pin_Memory_Board, Q1 TL431LP, SW1 SW_DIP_x08, U1 8259A-2, U10 74LS245, U11 74ALS573, U112 2764, U12 2764, U13 2764, U14 2764, U15 2764, U16 74ALS163, U17 74LS245, U18 74LS245, U19 74ALS573, U2 8259A-2, U20 74LS245, U21 74ALS573, U22 8237A, U23 8237A, U24 74ALS573, U25 74ALS573, U26 74LS244, U27 74LS245, U28 74LS243, U29 ATF16V8B, U3 74LS245, U30 74LS612, U31 ATF16V8B, U32 ATF16V8B, U33 74LS245, U34 74ALS573, U35 74ALS573, U37 74LS244, U38 ATF16V8B, U39 74LSA573, U4 74LS244, U40 74LS244, U41 74LS244, U44 8254, U45 8254, U46 ATF16V8B, U47 74LS125, U48 74LS125, U49 74LS138, U5 74LS590, U50 74LS175, U51 74LS244, U52 ATF16V8B, U53 74ALS08, U54 74ALS00, U55 74ALS04, U56 ATF22V10, U57 74LS273, U58 ATF22V10, U59 74F257BB, U6 MXO45HS-3C-14.3M, U61 74ALS74, U62 74LS51, U63 74ALS74, U64 ATF16V8B, U65 74F175, U66 74ALS00, U67 74ALS74, U68 ATF16V8B, U69 74F74, U7 74ALS74, U70 74ALS74, U71 74F00, U72 74ALS74, U73 74F08, U74 74F175, U75 74HC125, U76 I386DX_PGA, U77 MC146818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

Commit message: Update
Parts:
- C1, C100, C101, C114, C117, C2, C60, C97, C98: footprint (none) -> Capacitor_THT:C_Disc_D7.0mm_W2.5mm_P5.00mm; symbol Device:C -> 386_working:C
- C19, C9: footprint (none) -> Capacitor_THT:CP_Radial_D4.0mm_P2.00mm; symbol Device:C_Polarized -> 386_working:C_Polarized
- CR1, CR2, CR3: symbol Diode:1N914 -> 386_working:1N914
- E123: footprint (none) -> Connector_PinHeader_2.54mm:PinHeader_1x09_P2.54mm_Vertical; symbol Breadboarding:Conn_01x09_Pin_DP2 -> 386_working:Conn_01x09_Pin_DP2
- ER1, ER2: footprint (none) -> Connector_PinHeader_2.54mm:PinHeader_1x09_P2.54mm_Vertical; symbol Breadboarding:Conn_01x09_Pin_DP -> 386_working:Conn_01x09_Pin_DP
- F2: footprint (none) -> Fuse:Fuse_1206_3216Metric; symbol Device:Fuse_Small -> 386_working:Fuse_Small
- H2: footprint (none) -> Connector_PinHeader_2.54mm:PinHeader_1x02_P2.54mm_Vertical; symbol Switch:SW_SPST -> 386_working:SW_SPST
- J101: symbol Breadboarding:Conn_01x80_Pin_Memory_Board -> 386_working:Conn_01x80_Pin_Memory_Board_1
- J102: symbol Breadboarding:Bus_ISA_16bit -> 386_working:Bus_ISA_16bit
- J115, J118: footprint (none) -> Connector_PinHeader_2.54mm:PinHeader_1x04_P2.54mm_Vertical; symbol Connector:Conn_01x04_Socket -> 386_working:Conn_01x04_Socket
- J116: footprint (none) -> Connector_PinHeader_2.54mm:PinHeader_1x07_P2.54mm_Vertical; symbol Connector:Conn_01x07_Socket -> 386_working:Conn_01x07_Socket
- L1, L2, L3, L4, L6: footprint (none) -> Inductor_SMD:L_Panasonic_PCC-M0850M; symbol Device:FerriteBead_Small -> 386_working:FerriteBead_Small
- MRB4: symbol Device:R_Pack08_Split -> 386_working:R_Pack08_Split
- MRP1: footprint (none) -> Package_DIP:DIP-20_W7.62mm_Socket_LongPads; symbol Device:R_Pack10 -> 386_working:R_Pack10
- MRP5, MRP7, MRP8, MRP9, RP3, RP4, RP5, RP7: symbol Device:R_Network09 -> 386_working:R_Network09
- MRP6: symbol Device:R_Network10_Split -> 386_working:R_Network10_Split
- MU1, MU8, U61, U63, U67, U7, U70, U72, U81, U90: symbol Breadboarding:74ALS74 -> 386_working:74ALS74
- MU10, U53: symbol Breadboarding:74ALS08 -> 386_working:74ALS08
- MU11, MU12, MU14, MU6, U24, U25: symbol Breadboarding:74ALS573BBREVDP -> 386_working:74ALS573BBREVDP
- MU13, MU5: symbol Breadboarding:74F521DP -> 386_working:74F521DP
- MU15, MU16, MU17: symbol Breadboarding:74F158DP -> 386_working:74F158DP
- MU18: symbol Breadboarding:ATF16V8B_DP_D4RRAS -> 386_working:ATF16V8B_DP_D4RRAS
- MU19, MU24, MU3, MU50: symbol Breadboarding:74F32 -> 386_working:74F32
- MU2, U69, U79, U82, U83, U84: symbol Breadboarding:74F74 -> 386_working:74F74
- MU20, MU43: symbol 74xx:74LS20 -> 386_working:74LS20
- MU21, MU74, U65, U74, U89: symbol Breadboarding:74F175BB -> 386_working:74F175BB
- MU22: symbol Breadboarding:74ALS29827DP -> 386_working:74ALS29827DP
- MU25, U71: symbol Breadboarding:74F00 -> 386_working:74F00
- MU26, MU30, MU36, MU42: symbol Breadboarding:74F657DP -> 386_working:74F657DP
- MU31: symbol Breadboarding:51256-10DP -> 386_working:51256-10DP
- MU54, U26, U4: symbol Breadboarding:74LS244DP -> 386_working:74LS244DP
- MU59: symbol Breadboarding:ATF16V8B_DP_D4RCTLA -> 386_working:ATF16V8B_DP_D4RCTLA
- MU7: symbol Breadboarding:ATF16V8B_DP_RM32 -> 386_working:ATF16V8B_DP_RM32
- MU9: symbol Breadboarding:74F04 -> 386_working:74F04
- MU9: symbol 74xx:74LS04 -> 386_working:74LS04
- P101: symbol Breadboarding:Conn_01x80_Pin_Memory_Board -> 386_working:Conn_01x80_Pin_Memory_Board
- Q1: symbol Reference_Voltage:TL431LP -> 386_working:TL431LP
- R1, R10, R1000, R12, R13, R14, R15, R16, R17, R18, R19, R2, R20, R21, R22, R24, R25, R26, R28/9, R3, R30, R31, R33, R34, R35, R36, R37, R38, R39, R4, R40, R41, R42, R44, R5, R8, R999, RX1, RX2: footprint (none) -> Resistor_THT:R_Axial_DIN0207_L6.3mm_D2.5mm_P10.16mm_Horizontal; symbol Device:R -> 386_working:R
- RB4, RP6, RP8: symbol Device:R_Network08_Split -> 386_working:R_Network08_Split
- SW1: footprint (none) -> Button_Switch_THT:SW_DIP_SPSTx08_Slide_9.78x22.5mm_W7.62mm_P2.54mm; symbol Switch:SW_DIP_x08 -> 386_working:SW_DIP_x08
- U1, U2: symbol Breadboarding:8259A-2_DP_MIRROR -> 386_working:8259A-2_DP_MIRROR
- U10, U17, U18, U20, U3, U33, U8: symbol Breadboarding:74LS245 -> 386_working:74LS245
- U11: symbol Breadboarding:74LS573BBREV -> 386_working:74LS573BBREV_3
- U112, U14: symbol Breadboarding:2764DP -> 386_working:2764DP
- U12: symbol Breadboarding:74ALS1035 -> 386_working:74ALS1035_1
- U12: symbol Breadboarding:74ALS1035 -> 386_working:74ALS1035_2
- U13: symbol Breadboarding:74F175BB -> 386_working:74F175BB_1
- U13: symbol Breadboarding:2764DP -> 386_working:2764DP_2
- U14: symbol Breadboarding:74ALS02 -> 386_working:74ALS02_1
- U15: symbol Breadboarding:2764DP -> 386_working:2764DP_3
- U15: symbol Breadboarding:74ALS74 -> 386_working:74ALS74_1
- U16: symbol Breadboarding:74ALS163DP -> 386_working:74ALS163DP
- U19: symbol Breadboarding:74LS573BBREV -> 386_working:74LS573BBREV_2
- U21: symbol Breadboarding:74LS573BBREV -> 386_working:74LS573BBREV_4
- U22: symbol Breadboarding:intel_8237ADP -> 386_working:intel_8237ADP_1
- U23: symbol Breadboarding:intel_8237ADP -> 386_working:intel_8237ADP
- U27: symbol Breadboarding:74LS245DP -> 386_working:74LS245DP
- U28: symbol 74xx:74LS243 -> 386_working:74LS243
- U29: symbol Breadboarding:ATF16V8B_DP_D4SROMA -> 386_working:ATF16V8B_DP_D4SROMA
- U30: symbol Breadboarding:74ls612DP -> 386_working:74ls612DP
- U31: symbol Breadboarding:ATF16V8BB_DP_D4SCMDD -> 386_working:ATF16V8BB_DP_D4SCMDD
- U32: symbol Breadboarding:ATF16V8BB_DP_D4SDEND -> 386_working:ATF16V8BB_DP_D4SDEND
- U34: symbol Breadboarding:74LS573BBREV -> 386_working:74LS573BBREV_6
- U35: symbol Breadboarding:74LS573BBREV -> 386_working:74LS573BBREV_5
- U37: symbol Breadboarding:74LS244_2Halves -> 386_working:74LS244_2Halves
- U38: symbol Breadboarding:ATF16V8BB_DP_D4SADI -> 386_working:ATF16V8BB_DP_D4SADI
- U39: symbol Breadboarding:74LS573BBREV -> 386_working:74LS573BBREV
- U40, U41: symbol 74xx:74LS244 -> 386_working:74LS244
- U44: symbol Breadboarding:8254_dp -> 386_working:8254_dp
- U45: symbol Timer:8254 -> 386_working:8254
- U46: symbol Breadboarding:ATF16V8BB_DP_D4SCPYD -> 386_working:ATF16V8BB_DP_D4SCPYD
- U47, U48: symbol 74xx:74LS125 -> 386_working:74LS125
- U49: symbol Breadboarding:74LS138DP -> 386_working:74LS138DP
- U5: symbol 74xx:74LS590 -> 386_working:74LS590
- U50: symbol Breadboarding:74LS175DP -> 386_working:74LS175DP
- U51: symbol Breadboarding:74LS244DP2 -> 386_working:74LS244DP2
- U52: symbol Breadboarding:ATF16V8BB_DP_D4SNCP -> 386_working:ATF16V8BB_DP_D4SNCP
- U54, U66: symbol Breadboarding:74ALS00 -> 386_working:74ALS00
- U55: symbol Breadboarding:74ALS04 -> 386_working:74ALS04
- U56: symbol Breadboarding:ATF22V10_DP_D4STATB -> 386_working:ATF22V10_DP_D4STATB
- U57: symbol 74xx:74LS273 -> 386_working:74LS273
- U58: symbol Breadboarding:ATF22LV10_DP_D4SADOD -> 386_working:ATF22LV10_DP_D4SADOD
- U59: symbol Breadboarding:74F257BBDP -> 386_working:74F257BBDP
- U6: symbol Breadboarding:MXO45HS-3C-16M -> 386_working:MXO45HS-3C-16M
- U62: symbol 74xx:74LS51 -> 386_working:74LS51
- U64: symbol Breadboarding:ATF16V8BB_DP_D4SPPI -> 386_working:ATF16V8BB_DP_D4SPPI
- U66, U71: symbol 74xx:74LS00 -> 386_working:74LS00
- U68: symbol Breadboarding:ATF16V8BB_DP_D4SMSCD -> 386_working:ATF16V8BB_DP_D4SMSCD
- U7: symbol Breadboarding:74ALS74DP -> 386_working:74ALS74DP
- U73: symbol Breadboarding:74F08 -> 386_working:74F08
- U75: symbol Breadboarding:74HC125 -> 386_working:74HC125
- U76: symbol Breadboarding:I386DX_PGA -> 386_working:I386DX_PGA
- U77: symbol Breadboarding:MC146818DP -> 386_working:MC146818DP
- U78: symbol Breadboarding:INTEL_8042DP -> 386_working:INTEL_8042DP
- U85: symbol Breadboarding:MXO45HS-3C-32M -> 386_working:MXO45HS-3C-32M
- U86: symbol 4xxx:4069 -> 386_working:4069
- U88: symbol Breadboarding:74ALS02 -> 386_working:74ALS02_3
- U88: symbol Breadboarding:74ALS02 -> 386_working:74ALS02_4
- U88: symbol Breadboarding:74ALS02 -> 386_working:74ALS02
- U88: symbol Breadboarding:74ALS02 -> 386_working:74ALS02_2
- U9: symbol Breadboarding:74LS573BBREV -> 386_working:74LS573BBREV_1
- U91: symbol Breadboarding:74ALS1035_DP -> 386_working:74ALS1035_DP
- U92: symbol Breadboarding:74F11BB -> 386_working:74F11BB
- U92: symbol Breadboarding:74F11 -> 386_working:74F11
- U93: symbol Breadboarding:SN75477_DP -> 386_working:SN75477_DP
- Y2: symbol Device:Crystal -> 386_working:Crystal
Connections:
- net GND: now also R14.2, U59.14 (4A), U59.8 (GND), U76.A2 (VSS), U76.A6 (VSS), U76.A9 (VSS), U76.B1 (VSS), U76.B11 (VSS), U76.B14 (VSS), U76.B5 (VSS), U76.C11 (VSS), U76.F14 (VSS), U76.F2 (VSS), U76.F3 (VSS), U76.J12 (VSS), U76.J13 (VSS), U76.J2 (VSS), U76.J3 (VSS), U76.M10 (VSS), U76.M4 (VSS), U76.M8 (VSS), U76.N3 (VSS), U76.P14 (VSS), U76.P6 (VSS)

Commit message: Update
Parts:
- removed U12: 2764, Package_DIP:DIP-28_W15.24mm, symbol 386_working:74ALS1035_1
- removed unit 2 of U13
- removed unit 3 of U14
- removed unit 2 of U15
- removed unit 3 of U91
- added J10: AT POWER CONNECTOR, 386_draft:AT_power_connector, symbol Connector:Conn_01x12_Pin
- added J103: Bus_ISA_16bit, symbol 386_working:Bus_ISA_16bit
- U89: footprint (none) -> Package_DIP:DIP-16_W7.62mm_Socket_LongPads
- U91, U92: footprint (none) -> Package_SO:SOIC-14_3.9x8.7mm_P1.27mm
- U93: footprint (none) -> Package_DIP:DIP-8_W7.62mm_Socket_LongPads
- Y2: footprint (none) -> Crystal:Crystal_HC49-U_Vertical
- renumbered U112 to U12
Connections:
- net +12V: now also J10.3 (Pin_3), J103.B09 (+12V)
- net +5V: now also U91.14 (VCC), J10.10 (Pin_10), J10.11 (Pin_11), J10.12 (Pin_12), J103.B03 (+5V), J103.B29 (+5V), J103.D16 (+5V)
- net BALE: now also J103.B28 (BALE)
- net BCLK: now also J103.B20 (BCLK)
- net BUSRDY: now also J103.A10 (BUSRDY)
- net DMA: now also J103.A11 (AEN)
- net DRQ0: now also J103.D09 (DRQ0)
- net DRQ1: now also J103.B18 (DRQ1)
- net DRQ2: now also J103.B06 (DRQ2)
- net DRQ3: now also J103.B16 (DRQ3)
- net DRQ5: now also J103.D11 (DRQ5)
- net DRQ6: now also J103.D13 (DRQ6)
- net DRQ7: now also J103.D15 (DRQ7)
- net GND: now also U91.7 (GND), J10.5 (Pin_5), J10.6 (Pin_6), J10.7 (Pin_7), J10.8 (Pin_8), J103.B01 (GND), J103.B10 (GND), J103.B31 (GND), J103.D18 (GND)
- net IRQ10: now also J103.D03 (IRQ10)
- net IRQ11: now also J103.D04 (IRQ11)
- net IRQ12: now also J103.D05 (IRQ12)
- net IRQ14: now also J103.D07 (IRQ14)
- net IRQ15: now also J103.D06 (IRQ15)
- net IRQ3: now also J103.B25 (IRQ3)
- net IRQ4: now also J103.B24 (IRQ4)
- net IRQ5: now also J103.B23 (IRQ5)
- net IRQ6: now also J103.B22 (IRQ6)
- net IRQ7: now also J103.B21 (IRQ7)
- net IRQ9: now also J103.B04 (IRQ9)
- net KEYDAT: now also U91.6
- net LA17: now also J103.C08 (LA17)
- net LA18: now also J103.C07 (LA18)
- net LA19: now also J103.C06 (LA19)
- net LA20: now also J103.C05 (LA20)
- net LA21: now also J103.C04 (LA21)
- net LA22: now also J103.C03 (LA22)
- net LA23: now also J103.C02 (LA23)
- net OSC: now also J103.B30 (OSC)
- net P27: now also U91.5
- net PWROK: now also J10.1 (Pin_1)
- net RESDRV: now also J103.B02 (RESDRV)
- net SA0: now also J103.A31 (SA00)
- net SA1: now also J103.A30 (SA01)
- net SA10: now also J103.A21 (SA10)
- net SA11: now also J103.A20 (SA11)
- net SA12: now also J103.A19 (SA12)
- net SA13: now also J103.A18 (SA13)
- net SA16: now also J103.A15 (SA16), J103.A16 (SA15)
- net SA17: now also J103.A14 (SA17), J103.A17 (SA14)
- net SA18: now also J103.A13 (SA18)
- net SA19: now also J103.A12 (SA19)
- net SA2: now also J103.A29 (SA02)
- net SA3: now also J103.A28 (SA03)
- net SA4: now also J103.A27 (SA04)
- net SA5: now also J103.A26 (SA05)
- net SA6: now also J103.A25 (SA06)
- net SA7: now also J103.A24 (SA07)
- net SA8: now also J103.A23 (SA08)
- net SA9: now also J103.A22 (SA09)
- net SD0: now also J103.A09 (SD0)
- net SD1: now also J103.A08 (SD1)
- net SD10: now also J103.C13 (SD10)
- net SD11: now also J103.C14 (SD11)
- net SD12: now also J103.C15 (SD12)
- net SD13: now also J103.C16 (SD13)
- net SD14: now also J103.C17 (SD14)
- net SD15: now also J103.C18 (SD15)
- net SD2: now also J103.A07 (SD2)
- net SD3: now also J103.A06 (SD3)
- net SD4: now also J103.A05 (SD4)
- net SD5: now also J103.A04 (SD5)
- net SD6: now also J103.A03 (SD6)
- net SD7: now also J103.A02 (SD7)
- net SD8: now also J103.C11 (SD8)
- net SD9: now also J103.C12 (SD9)
- net T-C: now also J103.B27 (T/C)
- net ~{BHE}: now also J103.C01 (~{SBHE})
- net ~{DAK0}: now also J103.D08 (~{DACK0})
- net ~{DAK1}: now also J103.B17 (~{DAK1})
- net ~{DAK2}: now also J103.B26 (~{DAK2})
- net ~{DAK3}: now also J103.B15 (~{DAK3})
- net ~{DAK5}: now also J103.D10 (~{DACK5})
- net ~{DAK6}: now also J103.D12 (~{DACK6})
- net ~{DAK7}: now also J103.D14 (~{DACK7})
- net ~{GRAB}: now also J103.D17 (~{GRAB})
- net ~{IO16}: now also J103.D02 (~{IO16})
- net ~{IOCHK}: now also J103.A01 (~{IOCHK})
- net ~{IORC}: now also J103.B14 (~{IORC})
- net ~{IOWC}: now also J103.B13 (~{IOWC})
- net ~{M16}: now also J103.D01 (~{M16})
- net ~{MRDC}: now also J103.C09 (~{MRDC})
- net ~{MWTC}: now also J103.C10 (~{MWTC})
- net ~{NOWS}: now also J103.B08 (~{NOWS})
- net ~{REFRS}: now also J103.B19 (~{REFRESH})
- net ~{SMRDC}: now also J103.B12 (~{SMRDC})
- net ~{SMWTC}: now also J103.B11 (~{SMWTC})
- new net -12V: J10.4 (Pin_4), J103.B07 (-12V)
- new net -5V: J10.9 (Pin_9), J103.B05 (-5V)
- no-connect marks 85 -> 92
